File: 2-motor-controller/hardware/kicad/v00.01/Endstufe.kicad_sch (KiCad schematic)
At the start: 5 parts, among them J1 RF300, J2 12V Bordnetz, J5 Pumpe

Commit message: Motor-Controller: Hauptblatt nach Zweck gegliedert, Blatt Endstufe, eigene Bibliothek; Bauteilauswahl 00.20 / Stueckliste 00.16; 99-tools angelegt
Co-Authored-By: Claude Opus 5.5 <noreply@anthropic.com>
Parts:
- removed D1: 1.5KE20A, Diode_THT:D_DO-201AE_P15.24mm_Horizontal, symbol Diode:1.5KExxA
- removed D2: SB540, Diode_THT:D_DO-201AD_P15.24mm_Horizontal, symbol Device:D_Schottky
- removed J1: RF300, Connector_Phoenix_MSTB:PhoenixContact_MSTBA_2,5_2-G-5,08_1x02_P5.08mm_Horizontal, symbol Connector:Screw_Terminal_01x02
- removed J2: 12V Bordnetz, Connector_Phoenix_MSTB:PhoenixContact_MSTBA_2,5_2-G-5,08_1x02_P5.08mm_Horizontal, symbol Connector:Screw_Terminal_01x02
- removed J5: Pumpe, Connector_Phoenix_MSTB:PhoenixContact_MSTBA_2,5_2-G-5,08_1x02_P5.08mm_Horizontal, symbol Connector:Screw_Terminal_01x02
- added C10: 100n, Capacitor_THT:C_Disc_D7.5mm_W5.0mm_P5.00mm, symbol Device:C
- added C3: 1000u 35V, Capacitor_THT:CP_Radial_D12.5mm_P5.00mm, symbol Device:C_Polarized
- added D3: gelb A, LED_THT:LED_D3.0mm, symbol Device:LED
- added D4: gelb B, LED_THT:LED_D3.0mm, symbol Device:LED
- added J3, J4: Degson DG301, Motor-Controller:Degson_DG301-5.0-02P, symbol Connector:Screw_Terminal_01x02
- added J6: Temperaturfühler, Connector_Phoenix_MSTB:PhoenixContact_MSTBA_2,5_2-G-5,08_1x02_P5.08mm_Horizontal, symbol Connector:Screw_Terminal_01x02
- added R10: offen, Resistor_THT:R_Axial_DIN0207_L6.3mm_D2.5mm_P10.16mm_Horizontal, symbol Device:R
- added R11: 10k, Resistor_THT:R_Axial_DIN0207_L6.3mm_D2.5mm_P10.16mm_Horizontal, symbol Device:R
- added R12: 2k2, Resistor_THT:R_Axial_DIN0207_L6.3mm_D2.5mm_P10.16mm_Horizontal, symbol Device:R
- added U1: Pololu G2 18v25, Motor-Controller:Pololu_G2_18v25_Socket, symbol Motor-Controller:Pololu_G2_18v25
- added U2: ACS758LCB-050B-PFF-T, Sensor_Current:Allegro_CB_PFF, symbol Sensor_Current:ACS758xCB-050B-PFF
- added W1, W2, W3, W4: Leitung 20 mm 1,5 mm2, symbol Jumper:Jumper_2_Bridged
Connections:
- net +12V_LEISTUNG: now also J3.1 (Pin_1), W1.1 (A)
- net +3V3: now also R11.1
- net +5V: now also C10.1, U2.1 (VCC)
- net CS: now also U1.6 (CS)
- net DIR: now also U1.2 (DIR)
- net FLT: now also R11.2, U1.5 (~{FLT})
- net GND: now also C10.2, C3.2, J3.2 (Pin_2), J6.2 (Pin_2), R10.2, U1.1 (GND), U1.12 (C-), U1.9 (GND), U2.2 (GND), W2.1 (A)
- net HALL: now also U2.3 (VIOUT)
- net NTC: now also J6.1 (Pin_1)
- net PWM: now also U1.3 (PWM)
- net SLP: now also U1.4 (~{SLP})
- new net: J4.2 (Pin_2), U2.4 (IP+), W3.2 (B)
- new net: U1.15 (OUTA), W3.1 (A)
- new net: D3.2 (A), D4.1 (K), R12.2
- new net: U1.14 (GND), W2.2 (B)
- new net: R10.1, U1.10 (VREF)
- new net: U1.13 (VIN), W1.2 (B)
- new net: U1.16 (OUTB), W4.1 (A)
- new net KLEMME_A: R12.1, U2.5 (IP-)
- new net KLEMME_B: D3.1 (K), D4.2 (A), J4.1 (Pin_1), W4.2 (B)
- new net VM: C3.1, U1.11 (C+)
- no-connect marks 0 -> 2
Other:
- removed sheet 5V Elektronik
- removed sheet 5V PyPilot
- removed sheet Endstufe
- removed sheet RF300-Eingang
- note added: "Anzeige Pumpe (ohne Rechner)"
- note added: "D3 leuchtet: Pumpe Richtung A D4 leuchtet: Pumpe Richtung B R12: (14 V - ca. 2 V) / 2,2 kOhm = ca. 5,5 mA, 0,07 W (gerechnet)"
- note added: "J3 Degson DG301: kurze Leitungen zu Pololu VIN/GND (mind. 20 mm, höchstens 1,5 mm²)"
- note added: "J4 Degson DG301: kurze Leitungen von Pololu OUTA/OUTB. U2 (Hall-Sensor) in Ader A. KLEMME_A/B = Pumpenadern; die Pumpenklemme J5 sitzt im Hauptblatt am rechten Rand."
- note added: "J6 MSTBA 2,5/2: NTC unter der Befestigungsschraube des Pololu"
- note added: "Kondensatoren und Pololu-Klemmen zeigen zur Platine; Fläche darunter gesperrt. Am Pololu nur stecken und schrauben. C+ = VM hinter dem Verpolschutz: nie mit +12V verbinden. R10: Strombegrenzung 15 A, Wert offen (Kennlinie grob 17 kOhm). R11: FLT zieht nur nach Masse."
- note added: "Pololu G2 18v25 (Endstufe, umgedreht gesteckt)"
- note added: "Pumpenweg mit Strommessung"
- note added: "Temperaturfühler"
- note added: "Versorgung zum Pololu"
- note added: "W1-W4: kurze Leitungen zwischen den Pololu-Klemmen und J3/J4 (mind. 20 mm, max. 1,5 mm²), nicht auf der Platine. Unter den Pololu-Klemmen nur Hilfslötaugen (Pololu-Bauform, Unterseite)."
- note removed: "12 V vom Bordnetz (2,5 mm², Sicherung 20 A im Schiff) J2: Phoenix MSTBA 2,5/2 D1: Überspannungsschutz, klemmt 27,7 V (Endstufe verträgt 30 V) +12V_LEISTUNG: über J3 und kurze Leitungen zum Pololu VIN D2: Verpolschutz nur für den Elektronikzweig (+12V)"
- note removed: "Bordnetz-Eingang"
- note removed: "J5 MSTBA 2,5/2 zur Pumpe RPU160 Ader A über den Hall-Sensor (Blatt Endstufe)"
- note removed: "Pumpe antreiben"
- note removed: "Ruderlage"
- note removed: "Steuerung"
- note removed: "Verbindung zum Steuerhaus"
- note removed: "zum RF300 (Kabel max. 3 m, geschirmt, Schirm an Masse) J1: Phoenix MSTBA 2,5 (wie RF300-Interface)"

Commit message: Motor-Controller: alle Blaetter nach den Zeichenregeln (Rahmen, Gruppen), 5-V-Zweig mit 2 x 4,7 uF, Titelfelder Version 00.01; Pruefung gegen Blockschaltbild 78/78
Co-Authored-By: Claude Opus 5.5 <noreply@anthropic.com>
Other:
- company: (none) -> SuAn-Autopilot-Projekt
- title: (none) -> Motor-Controller V2.0 – Endstufe
Changed lines of the file:
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@@
 	(generator_version "10.0")
 	(paper "A4")
+	(title_block
+		(title "Motor-Controller V2.0 – Endstufe")
+		(date "2026-10-09")
+		(rev "00.01")
+		(company "SuAn-Autopilot-Projekt")
+	)
 	(rectangle
 		(start 177.8 88.9)
@@
 	(wire
 		(pts
-			(xy 78.74 53.34) (xy 109.22 53.34)
+			(xy 83.82 53.34) (xy 109.22 53.34)
 		)
 		(stroke
@@
 	(wire
 		(pts
-			(xy 78.74 55.88) (xy 109.22 55.88)
+			(xy 83.82 55.88) (xy 109.22 55.88)
 		)
 		(stroke
@@
 	(wire
 		(pts
-			(xy 78.74 58.42) (xy 109.22 58.42)
+			(xy 83.82 58.42) (xy 109.22 58.42)
 		)
 		(stroke
@@
 	(hierarchical_label "SLP"
 		(shape input)
-		(at 78.74 58.42 180)
+		(at 83.82 58.42 180)
 		(effects
 			(font
@@
 	(hierarchical_label "PWM"
 		(shape input)
-		(at 78.74 55.88 180)
+		(at 83.82 55.88 180)
 		(effects
 			(font
@@
 	(hierarchical_label "DIR"
 		(shape input)
-		(at 78.74 53.34 180)
-		(effects
-			(font
+		(at 83.82 53.34 180)
+		(effects
+			(font

Commit message: Motor-Controller: Bauteile vollstaendig gewaehlt, Strombegrenzung in Software
- Leisten Wuerth WR-PHD (Buchse 8,5 mm, Stift), Stehbolzen M2 x 12, Taster E-Switch TL1105NF250Q (Winkel),
  Referenz LM4040AIZ-2.5 (+-0,1 %), Sicherungshalter Schurter 0031.8201, Leuchtdioden Dialight 551 (Winkel, rechte Kante)
- Strombegrenzung in der Software (Hall-Sensor), R10 an VREF nicht bestueckt
- Display-Beleuchtung aus +5 V ueber R610 220 Ohm; Vorwiderstand gruen 270 Ohm
- Selbsttest laeuft staendig ohne Ruderbewegung; WLAN ohne aeussere Antenne
- Pruefskript pruefung_blockschaltbild.py im Projekt: 80/80, ERC 0 Fehler
- Bauteilauswahl 00.22, Stueckliste 00.18, Anforderungen 00.11, Blockschaltbild 00.06, Messgeraet 00.03,
  Systembeschreibung, TODO, CHRONIK (Lehre Schaltplan), CLAUDE.md (Arbeitsweg KiCad)

Co-Authored-By: Claude Opus 5.5 <noreply@anthropic.com>
Parts:
- R10: value offen -> nicht bestückt; now not fitted
Other:
- note added: "Kondensatoren und Pololu-Klemmen zeigen zur Platine; Fläche darunter gesperrt. Am Pololu nur stecken und schrauben. C+ = VM hinter dem Verpolschutz: nie mit +12V verbinden. R10: nicht bestückt, Strombegrenzung in der Software. R11: FLT zieht nur nach Masse."
- note removed: "Kondensatoren und Pololu-Klemmen zeigen zur Platine; Fläche darunter gesperrt. Am Pololu nur stecken und schrauben. C+ = VM hinter dem Verpolschutz: nie mit +12V verbinden. R10: Strombegrenzung 15 A, Wert offen (Kennlinie grob 17 kOhm). R11: FLT zieht nur nach Masse."
Changed lines of the file:
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@@
 		)
 	)
-	(text "Kondensatoren und Pololu-Klemmen zeigen zur Platine;\nFläche darunter gesperrt. Am Pololu nur stecken und schrauben.\nC+ = VM hinter dem Verpolschutz: nie mit +12V verbinden.\nR10: Strombegrenzung 15 A, Wert offen (Kennlinie grob 17 kOhm).\nR11: FLT zieht nur nach Masse."
+	(text "Kondensatoren und Pololu-Klemmen zeigen zur Platine;\nFläche darunter gesperrt. Am Pololu nur stecken und schrauben.\nC+ = VM hinter dem Verpolschutz: nie mit +12V verbinden.\nR10: nicht bestückt, Strombegrenzung in der Software.\nR11: FLT zieht nur nach Masse."
 		(exclude_from_sim no)
 		(at 74.93 93.98 0)
@@
 		(on_board yes)
 		(in_pos_files yes)
-		(dnp no)
+		(dnp yes)
 		(property "Reference" "R10"
-			(at 92.71 69.85 0)
-			(show_name no)
-			(do_not_autoplace no)
-			(effects
-				(font
-					(size 1.27 1.27)
-				)
-				(justify left)
-			)
-		)
-		(property "Value" "offen"
-			(at 92.71 72.39 0)
-			(show_name no)
-			(do_not_autoplace no)
-			(effects
-				(font
-					(size 1.27 1.27)
-				)
-				(justify left)
-			)
-		)
+			(at 99.06 69.85 0)
+			(show_name no)
+			(do_not_autoplace no)
+			(effects
+				(font
+					(size 1.27 1.27)
+				)
+				(justify right)
+			)
+		)
+		(property "Value" "nicht bestückt"
+			(at 99.06 72.39 0)
+			(show_name no)
+			(do_not_autoplace no)
+			(effects
+				(font
+					(size 1.27 1.27)
+				)
+				(justify right)
+			)
+		)

Commit message: Motor-Controller: Loetbilder zugeordnet (eigene: Dialight 551, TL1105, KEMET C320, Display-Leiste), Platine 150 x 130 mm mit allen 94 Teilen angeordnet - Bauteilauswahl 00.23, Anforderungen 00.11, Stueckliste 00.19
Co-Authored-By: Claude Opus 5.5 <noreply@anthropic.com>
Parts:
- C10: footprint Capacitor_THT:C_Disc_D7.5mm_W5.0mm_P5.00mm -> Motor-Controller:C_KEMET_C320_L5.1mm_W4.1mm_P2.54mm
- D3, D4: footprint LED_THT:LED_D3.0mm -> Motor-Controller:LED_Dialight_551_RightAngle
Changed lines of the file:
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@@
 			)
 		)
-		(property "Footprint" "Capacitor_THT:C_Disc_D7.5mm_W5.0mm_P5.00mm"
+		(property "Footprint" "Motor-Controller:C_KEMET_C320_L5.1mm_W4.1mm_P2.54mm"
 			(at 239.725 40.64 0)
 			(hide yes)
@@
 			)
 		)
-		(property "Footprint" "LED_THT:LED_D3.0mm"
+		(property "Footprint" "Motor-Controller:LED_Dialight_551_RightAngle"
 			(at 233.68 105.41 0)
 			(hide yes)
@@
 			)
 		)
-		(property "Footprint" "LED_THT:LED_D3.0mm"
+		(property "Footprint" "Motor-Controller:LED_Dialight_551_RightAngle"
 			(at 220.98 105.41 0)
 			(hide yes)

Commit message: Motor-Controller: J6 feste Degson DG301 statt steckbarer MSTBA; J7 neue Belegung (1 MCY, 2 MCZ, 3 MCB, 4 MCA, 5 RAA, 6 RAB, 7 GND, 8 +5V), J8 entfaellt - Bauteilauswahl 00.24, Stueckliste 00.20, Pruefskript 00.02
Co-Authored-By: Claude Opus 5.5 <noreply@anthropic.com>
Parts:
- J6: footprint Connector_Phoenix_MSTB:PhoenixContact_MSTBA_2,5_2-G-5,08_1x02_P5.08mm_Horizontal -> Motor-Controller:Degson_DG301-5.0-02P
Other:
- note added: "J6 Degson DG301: NTC unter der Befestigungsschraube des Pololu"
- note removed: "J6 MSTBA 2,5/2: NTC unter der Befestigungsschraube des Pololu"
Changed lines of the file:
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@@
 		)
 	)
-	(text "J6 MSTBA 2,5/2: NTC unter der\nBefestigungsschraube des Pololu"
+	(text "J6 Degson DG301: NTC unter der\nBefestigungsschraube des Pololu"
 		(exclude_from_sim no)
 		(at 13.97 93.98 0)
@@
 			)
 		)
-		(property "Footprint" "Connector_Phoenix_MSTB:PhoenixContact_MSTBA_2,5_2-G-5,08_1x02_P5.08mm_Horizontal"
+		(property "Footprint" "Motor-Controller:Degson_DG301-5.0-02P"
 			(at 25.4 78.74 0)
 			(hide yes)
