File: 2-motor-controller/hardware/kicad/v00.01/Messwerterfassung.kicad_sch (KiCad schematic)
At the start: 25 parts, among them U301 MCP3208, U302 LM4040DIZ-2.5

Commit message: Motor-Controller: alle Blaetter nach den Zeichenregeln (Rahmen, Gruppen), 5-V-Zweig mit 2 x 4,7 uF, Titelfelder Version 00.01; Pruefung gegen Blockschaltbild 78/78
Co-Authored-By: Claude Opus 5.5 <noreply@anthropic.com>
Other:
- company: (none) -> SuAn-Autopilot-Projekt
- title: (none) -> Motor-Controller V2.0 – Messwerterfassung
Changed lines of the file:
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@@
 	(generator_version "10.0")
 	(paper "A4")
+	(title_block
+		(title "Motor-Controller V2.0 – Messwerterfassung")
+		(date "2026-10-09")
+		(rev "00.01")
+		(company "SuAn-Autopilot-Projekt")
+	)
 	(rectangle
 		(start 12.7 17.78)

Commit message: Motor-Controller: Bauteile vollstaendig gewaehlt, Strombegrenzung in Software
- Leisten Wuerth WR-PHD (Buchse 8,5 mm, Stift), Stehbolzen M2 x 12, Taster E-Switch TL1105NF250Q (Winkel),
  Referenz LM4040AIZ-2.5 (+-0,1 %), Sicherungshalter Schurter 0031.8201, Leuchtdioden Dialight 551 (Winkel, rechte Kante)
- Strombegrenzung in der Software (Hall-Sensor), R10 an VREF nicht bestueckt
- Display-Beleuchtung aus +5 V ueber R610 220 Ohm; Vorwiderstand gruen 270 Ohm
- Selbsttest laeuft staendig ohne Ruderbewegung; WLAN ohne aeussere Antenne
- Pruefskript pruefung_blockschaltbild.py im Projekt: 80/80, ERC 0 Fehler
- Bauteilauswahl 00.22, Stueckliste 00.18, Anforderungen 00.11, Blockschaltbild 00.06, Messgeraet 00.03,
  Systembeschreibung, TODO, CHRONIK (Lehre Schaltplan), CLAUDE.md (Arbeitsweg KiCad)

Co-Authored-By: Claude Opus 5.5 <noreply@anthropic.com>
Parts:
- U302: value LM4040DIZ-2.5 -> LM4040AIZ-2.5
Changed lines of the file:
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@@
 			)
 		)
-		(property "Value" "LM4040DIZ-2.5"
+		(property "Value" "LM4040AIZ-2.5"
 			(at 216.53 62.23 0)
 			(show_name no)

Commit message: Motor-Controller: Loetbilder zugeordnet (eigene: Dialight 551, TL1105, KEMET C320, Display-Leiste), Platine 150 x 130 mm mit allen 94 Teilen angeordnet - Bauteilauswahl 00.23, Anforderungen 00.11, Stueckliste 00.19
Co-Authored-By: Claude Opus 5.5 <noreply@anthropic.com>
Parts:
- C301, C302, C303, C304, C306: footprint (none) -> Motor-Controller:C_KEMET_C320_L5.1mm_W4.1mm_P2.54mm
- C305: footprint (none) -> Capacitor_THT:C_Rect_L7.2mm_W4.5mm_P5.00mm_FKS2_FKP2_MKS2_MKP2
- D301, D302, D303, D304, D305, D306: footprint Diode_THT:D_DO-35_SOD27_P7.62mm_Horizontal -> Diode_THT:D_DO-34_SOD68_P7.62mm_Horizontal
- R301, R302, R303, R304, R305, R306, R307, R308, R309, R310, R311: footprint (none) -> Resistor_THT:R_Axial_DIN0207_L6.3mm_D2.5mm_P10.16mm_Horizontal
- U301: footprint (none) -> Package_DIP:DIP-16_W7.62mm_Socket
Changed lines of the file:
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@@
 			)
 		)
-		(property "Footprint" ""
+		(property "Footprint" "Resistor_THT:R_Axial_DIN0207_L6.3mm_D2.5mm_P10.16mm_Horizontal"
 			(at 35.56 35.56 0)
 			(hide yes)
@@
 			)
 		)
-		(property "Footprint" ""
+		(property "Footprint" "Resistor_THT:R_Axial_DIN0207_L6.3mm_D2.5mm_P10.16mm_Horizontal"
 			(at 45.72 43.18 0)
 			(hide yes)
@@
 			)
 		)
-		(property "Footprint" ""
+		(property "Footprint" "Resistor_THT:R_Axial_DIN0207_L6.3mm_D2.5mm_P10.16mm_Horizontal"
 			(at 55.88 50.8 0)
 			(hide yes)
@@
 			)
 		)
-		(property "Footprint" ""
+		(property "Footprint" "Motor-Controller:C_KEMET_C320_L5.1mm_W4.1mm_P2.54mm"
 			(at 68.58 50.8 0)
 			(hide yes)
@@
 			)
 		)
-		(property "Footprint" "Diode_THT:D_DO-35_SOD27_P7.62mm_Horizontal"
+		(property "Footprint" "Diode_THT:D_DO-34_SOD68_P7.62mm_Horizontal"
 			(at 81.28 35.56 0)
 			(hide yes)
@@
 			)
 		)
-		(property "Footprint" "Diode_THT:D_DO-35_SOD27_P7.62mm_Horizontal"
+		(property "Footprint" "Diode_THT:D_DO-34_SOD68_P7.62mm_Horizontal"
 			(at 81.28 50.8 0)
 			(hide yes)
@@
 			)
 		)
-		(property "Footprint" ""
+		(property "Footprint" "Resistor_THT:R_Axial_DIN0207_L6.3mm_D2.5mm_P10.16mm_Horizontal"
 			(at 45.72 83.82 0)
 			(hide yes)
@@
 			)
 		)
-		(property "Footprint" ""
+		(property "Footprint" "Resistor_THT:R_Axial_DIN0207_L6.3mm_D2.5mm_P10.16mm_Horizontal"
 			(at 55.88 91.44 0)
 			(hide yes)
@@
 			)
 		)
-		(property "Footprint" ""
+		(property "Footprint" "Motor-Controller:C_KEMET_C320_L5.1mm_W4.1mm_P2.54mm"
 			(at 68.58 91.44 0)
 			(hide yes)
@@
 			)
 		)
-		(property "Footprint" "Diode_THT:D_DO-35_SOD27_P7.62mm_Horizontal"
+		(property "Footprint" "Diode_THT:D_DO-34_SOD68_P7.62mm_Horizontal"
 			(at 81.28 76.2 0)
 			(hide yes)
@@
 			)
 		)
-		(property "Footprint" "Diode_THT:D_DO-35_SOD27_P7.62mm_Horizontal"
+		(property "Footprint" "Diode_THT:D_DO-34_SOD68_P7.62mm_Horizontal"
 			(at 81.28 91.44 0)
 			(hide yes)
@@
 			)
 		)
-		(property "Footprint" ""
+		(property "Footprint" "Resistor_THT:R_Axial_DIN0207_L6.3mm_D2.5mm_P10.16mm_Horizontal"
 			(at 45.72 149.86 0)
 			(hide yes)
@@
 			)
 		)
-		(property "Footprint" ""
+		(property "Footprint" "Resistor_THT:R_Axial_DIN0207_L6.3mm_D2.5mm_P10.16mm_Horizontal"
 			(at 55.88 157.48 0)
 			(hide yes)
@@
 			)
 		)
-		(property "Footprint" ""
+		(property "Footprint" "Motor-Controller:C_KEMET_C320_L5.1mm_W4.1mm_P2.54mm"
 			(at 68.58 157.48 0)
 			(hide yes)
@@
 			)
 		)
-		(property "Footprint" "Diode_THT:D_DO-35_SOD27_P7.62mm_Horizontal"
+		(property "Footprint" "Diode_THT:D_DO-34_SOD68_P7.62mm_Horizontal"
 			(at 81.28 142.24 0)
 			(hide yes)
@@
 			)
 		)
-		(property "Footprint" "Diode_THT:D_DO-35_SOD27_P7.62mm_Horizontal"
+		(property "Footprint" "Diode_THT:D_DO-34_SOD68_P7.62mm_Horizontal"
 			(at 81.28 157.48 0)
 			(hide yes)
@@
 			)
 		)
-		(property "Footprint" ""
+		(property "Footprint" "Resistor_THT:R_Axial_DIN0207_L6.3mm_D2.5mm_P10.16mm_Horizontal"
 			(at 129.54 43.18 0)
 			(hide yes)
@@
 			)
 		)
-		(property "Footprint" ""
+		(property "Footprint" "Resistor_THT:R_Axial_DIN0207_L6.3mm_D2.5mm_P10.16mm_Horizontal"
 			(at 139.7 50.8 0)
 			(hide yes)
@@
 			)
 		)
-		(property "Footprint" ""
+		(property "Footprint" "Resistor_THT:R_Axial_DIN0207_L6.3mm_D2.5mm_P10.16mm_Horizontal"
 			(at 129.54 76.2 0)
 			(hide yes)
@@
 			)
 		)
-		(property "Footprint" ""
+		(property "Footprint" "Motor-Controller:C_KEMET_C320_L5.1mm_W4.1mm_P2.54mm"
 			(at 139.7 91.44 0)
 			(hide yes)
@@
 			)
 		)
-		(property "Footprint" ""
+		(property "Footprint" "Package_DIP:DIP-16_W7.62mm_Socket"
 			(at 236.22 76.2 0)
 			(hide yes)
@@
 			)
 		)
-		(property "Footprint" ""
+		(property "Footprint" "Resistor_THT:R_Axial_DIN0207_L6.3mm_D2.5mm_P10.16mm_Horizontal"
 			(at 198.12 40.64 0)
 			(hide yes)
@@
 			)
 		)
-		(property "Footprint" ""
+		(property "Footprint" "Capacitor_THT:C_Rect_L7.2mm_W4.5mm_P5.00mm_FKS2_FKP2_MKS2_MKP2"
 			(at 198.12 53.34 0)
 			(hide yes)
@@
 			)
 		)
-		(property "Footprint" ""
+		(property "Footprint" "Motor-Controller:C_KEMET_C320_L5.1mm_W4.1mm_P2.54mm"
 			(at 248.92 50.8 0)
 			(hide yes)
