File: 2-motor-controller/hardware/kicad/v00.01/Motor-Controller.kicad_pcb (KiCad board)
At the start: 2 copper layers, 0 parts

Commit message: Motor-Controller: Loetbilder zugeordnet (eigene: Dialight 551, TL1105, KEMET C320, Display-Leiste), Platine 150 x 130 mm mit allen 94 Teilen angeordnet - Bauteilauswahl 00.23, Anforderungen 00.11, Stueckliste 00.19
Co-Authored-By: Claude Opus 5.5 <noreply@anthropic.com>
Parts:
- added C1: 100n, Motor-Controller:C_KEMET_C320_L5.1mm_W4.1mm_P2.54mm, F.Cu at (63.4, 128.5)
- added C10: 100n, Motor-Controller:C_KEMET_C320_L5.1mm_W4.1mm_P2.54mm, F.Cu at (118.3, 137.5)
- added C101: 4u7 50V, Motor-Controller:C_KEMET_C320_L5.1mm_W4.1mm_P2.54mm, F.Cu at (87.6, 77.3)
- added C102: 4u7 50V, Motor-Controller:C_KEMET_C320_L5.1mm_W4.1mm_P2.54mm, F.Cu at (94.7, 77.3)
- added C103: 4u7 50V, Motor-Controller:C_KEMET_C320_L5.1mm_W4.1mm_P2.54mm, F.Cu at (101.9, 77.3)
- added C2: 10n, Motor-Controller:C_KEMET_C320_L5.1mm_W4.1mm_P2.54mm, F.Cu at (70.6, 128.5)
- added C201: 4u7 50V, Motor-Controller:C_KEMET_C320_L5.1mm_W4.1mm_P2.54mm, F.Cu at (113.2, 83.5)
- added C202: 4u7 50V, Motor-Controller:C_KEMET_C320_L5.1mm_W4.1mm_P2.54mm, F.Cu at (120.4, 83.5)
- added C203: 4u7 50V, Motor-Controller:C_KEMET_C320_L5.1mm_W4.1mm_P2.54mm, F.Cu at (90.6, 148.3)
- added C3: 1000u 35V, Capacitor_THT:CP_Radial_D12.5mm_P5.00mm, F.Cu at (142.5, 61.9)
- added C301: 680n, Motor-Controller:C_KEMET_C320_L5.1mm_W4.1mm_P2.54mm, F.Cu at (124.2, 118.7)
- added C302: 680n, Motor-Controller:C_KEMET_C320_L5.1mm_W4.1mm_P2.54mm, F.Cu at (131.4, 118.7)
- added C303: 100n, Motor-Controller:C_KEMET_C320_L5.1mm_W4.1mm_P2.54mm, F.Cu at (138.6, 118.7)
- added C304: 100n, Motor-Controller:C_KEMET_C320_L5.1mm_W4.1mm_P2.54mm, F.Cu at (145.7, 118.7)
- added C305: 1u, Capacitor_THT:C_Rect_L7.2mm_W4.5mm_P5.00mm_FKS2_FKP2_MKS2_MKP2, F.Cu at (152.7, 118.9)
- added C306: 100n, Motor-Controller:C_KEMET_C320_L5.1mm_W4.1mm_P2.54mm, F.Cu at (162.2, 118.7)
- added C401: 100n, Motor-Controller:C_KEMET_C320_L5.1mm_W4.1mm_P2.54mm, F.Cu at (122.8, 125.3)
- added C501: 100n, Motor-Controller:C_KEMET_C320_L5.1mm_W4.1mm_P2.54mm, F.Cu at (155.1, 125.3)
- added C601: 100n, Motor-Controller:C_KEMET_C320_L5.1mm_W4.1mm_P2.54mm, F.Cu at (111.6, 103.3)
- added D1: 1.5KE20A, Diode_THT:D_DO-201AE_P15.24mm_Horizontal, F.Cu at (87.6, 55.9)
- added D101: rot, Motor-Controller:LED_Dialight_551_RightAngle, F.Cu at (87.2, 44.4)
- added D2: SB540, Diode_THT:D_DO-201AD_P15.24mm_Horizontal, F.Cu at (107.8, 55.9)
- added D201: rot, Motor-Controller:LED_Dialight_551_RightAngle, F.Cu at (146.5, 44.4)
- added D3: gelb A, Motor-Controller:LED_Dialight_551_RightAngle, F.Cu at (44.4, 98.9)
- added D301: BAT85, Diode_THT:D_DO-34_SOD68_P7.62mm_Horizontal, F.Cu at (131.6, 112.9)
- added D302: BAT85, Diode_THT:D_DO-34_SOD68_P7.62mm_Horizontal, F.Cu at (142.8, 112.9)
- added D303: BAT85, Diode_THT:D_DO-34_SOD68_P7.62mm_Horizontal, F.Cu at (154.0, 112.9)
- added D304: BAT85, Diode_THT:D_DO-34_SOD68_P7.62mm_Horizontal, F.Cu at (90.0, 117.4)
- added D305: BAT85, Diode_THT:D_DO-34_SOD68_P7.62mm_Horizontal, F.Cu at (101.3, 117.4)
- added D306: BAT85, Diode_THT:D_DO-34_SOD68_P7.62mm_Horizontal, F.Cu at (112.5, 117.4)
- added D4: gelb B, Motor-Controller:LED_Dialight_551_RightAngle, F.Cu at (44.4, 106.5)
- added D601: grün Betrieb, Motor-Controller:LED_Dialight_551_RightAngle, F.Cu at (44.4, 76.0)
- added D602: rot Störung, Motor-Controller:LED_Dialight_551_RightAngle, F.Cu at (44.4, 83.6)
- added D603: blau WLAN, Motor-Controller:LED_Dialight_551_RightAngle, F.Cu at (44.4, 91.2)
- added DS601: LCD 12864B ST7920, Motor-Controller:LCD_12864B_Socket, F.Cu at (141.8, 163.5)
- added F101: 2A T, Fuse:Fuseholder_Cylinder-5x20mm_Schurter_0031_8201_Horizontal_Open, F.Cu at (93.3, 45.7)
- added F201: 2A T, Fuse:Fuseholder_Cylinder-5x20mm_Schurter_0031_8201_Horizontal_Open, F.Cu at (120.3, 45.7)
- added J1: RF300, Connector_Phoenix_MSTB:PhoenixContact_MSTBA_2,5_2-G-5,08_1x02_P5.08mm_Horizontal, F.Cu at (50.3, 61.6)
- added J2: 12V Bordnetz, Connector_Phoenix_MSTB:PhoenixContact_MSTBA_2,5_2-G-5,08_1x02_P5.08mm_Horizontal, F.Cu at (50.3, 47.1)
- added J3: Degson DG301, Motor-Controller:Degson_DG301-5.0-02P, F.Cu at (156.4, 84.8)
- added J4: Degson DG301, Motor-Controller:Degson_DG301-5.0-02P, F.Cu at (168.4, 84.8)
- added J5: Pumpe, Connector_Phoenix_MSTB:PhoenixContact_MSTBA_2,5_2-G-5,08_1x02_P5.08mm_Horizontal, F.Cu at (179.7, 52.2)
- added J6: Temperaturfühler, Connector_Phoenix_MSTB:PhoenixContact_MSTBA_2,5_2-G-5,08_1x02_P5.08mm_Horizontal, F.Cu at (90.1, 62.9)
- added J7: Steuerhaus RS422, Connector_Phoenix_MSTB:PhoenixContact_MSTBA_2,5_8-G-5,08_1x08_P5.08mm_Horizontal, F.Cu at (179.7, 111.6)
- added J8: Steuerhaus 5V, Connector_Phoenix_MSTB:PhoenixContact_MSTBA_2,5_2-G-5,08_1x02_P5.08mm_Horizontal, F.Cu at (179.7, 66.7)
- added L101: 10uH 2,7A, Inductor_THT:L_Radial_D10.0mm_P5.00mm_Fastron_07P, F.Cu at (103.6, 65.7)
- added L201: 10uH 2,7A, Inductor_THT:L_Radial_D10.0mm_P5.00mm_Fastron_07P, F.Cu at (88.8, 86.4)
- added Q3: BC337, Package_TO_SOT_THT:TO-92_Inline, F.Cu at (49.5, 135.2)
- added Q601: BC337, Package_TO_SOT_THT:TO-92_Inline, F.Cu at (49.5, 164.4)
- added Q602: BC337, Package_TO_SOT_THT:TO-92_Inline, F.Cu at (56.6, 164.4)
- added Q603: BC337, Package_TO_SOT_THT:TO-92_Inline, F.Cu at (63.6, 164.4)
- added Q604: BC337, Package_TO_SOT_THT:TO-92_Inline, F.Cu at (70.7, 164.4)
- added R1: 220R 2W, Resistor_THT:R_Axial_DIN0617_L17.0mm_D6.0mm_P20.32mm_Horizontal, F.Cu at (49.5, 116.8)
- added R10: nicht bestückt, Resistor_THT:R_Axial_DIN0207_L6.3mm_D2.5mm_P10.16mm_Horizontal, F.Cu at (90.1, 136.7)
- added R101: 4k7, Resistor_THT:R_Axial_DIN0207_L6.3mm_D2.5mm_P10.16mm_Horizontal, F.Cu at (108.6, 76.5)
- added R11: 10k, Resistor_THT:R_Axial_DIN0207_L6.3mm_D2.5mm_P10.16mm_Horizontal, F.Cu at (103.9, 136.7)
- added R12: 2k2, Resistor_THT:R_Axial_DIN0207_L6.3mm_D2.5mm_P10.16mm_Horizontal, F.Cu at (56.1, 133.9)
- added R201: 4k7, Resistor_THT:R_Axial_DIN0207_L6.3mm_D2.5mm_P10.16mm_Horizontal, F.Cu at (97.1, 147.5)
- added R301: 100k, Resistor_THT:R_Axial_DIN0207_L6.3mm_D2.5mm_P10.16mm_Horizontal, F.Cu at (118.3, 102.5)
- added R302: 100k 1%, Resistor_THT:R_Axial_DIN0207_L6.3mm_D2.5mm_P10.16mm_Horizontal, F.Cu at (132.1, 102.5)
- added R303: 18k 1%, Resistor_THT:R_Axial_DIN0207_L6.3mm_D2.5mm_P10.16mm_Horizontal, F.Cu at (146.0, 102.5)
- added R304: 100k 1%, Resistor_THT:R_Axial_DIN0207_L6.3mm_D2.5mm_P10.16mm_Horizontal, F.Cu at (90.1, 108.7)
- added R305: 18k 1%, Resistor_THT:R_Axial_DIN0207_L6.3mm_D2.5mm_P10.16mm_Horizontal, F.Cu at (103.9, 108.7)
- added R306: 100k 1%, Resistor_THT:R_Axial_DIN0207_L6.3mm_D2.5mm_P10.16mm_Horizontal, F.Cu at (117.8, 108.7)
- added R307: 18k 1%, Resistor_THT:R_Axial_DIN0207_L6.3mm_D2.5mm_P10.16mm_Horizontal, F.Cu at (131.6, 108.7)
- added R308: 10k 1%, Resistor_THT:R_Axial_DIN0207_L6.3mm_D2.5mm_P10.16mm_Horizontal, F.Cu at (145.5, 108.7)
- added R309: 10k 1%, Resistor_THT:R_Axial_DIN0207_L6.3mm_D2.5mm_P10.16mm_Horizontal, F.Cu at (90.1, 113.3)
- added R310: 12k 1%, Resistor_THT:R_Axial_DIN0207_L6.3mm_D2.5mm_P10.16mm_Horizontal, F.Cu at (103.9, 113.3)
- added R311: 1k, Resistor_THT:R_Axial_DIN0207_L6.3mm_D2.5mm_P10.16mm_Horizontal, F.Cu at (117.8, 113.3)
- added R4: 22k, Resistor_THT:R_Axial_DIN0207_L6.3mm_D2.5mm_P10.16mm_Horizontal, F.Cu at (49.1, 123.2)
- added R401: 120 1%, Resistor_THT:R_Axial_DIN0207_L6.3mm_D2.5mm_P10.16mm_Horizontal, F.Cu at (108.5, 124.5)
- added R5: 10k, Resistor_THT:R_Axial_DIN0207_L6.3mm_D2.5mm_P10.16mm_Horizontal, F.Cu at (62.9, 123.2)
- added R501: 120 1%, Resistor_THT:R_Axial_DIN0207_L6.3mm_D2.5mm_P10.16mm_Horizontal, F.Cu at (140.8, 124.5)
- added R6: 1k, Resistor_THT:R_Axial_DIN0207_L6.3mm_D2.5mm_P10.16mm_Horizontal, F.Cu at (49.1, 127.8)
- added R601: 10k, Resistor_THT:R_Axial_DIN0207_L6.3mm_D2.5mm_P10.16mm_Horizontal, F.Cu at (49.1, 140.3)
- added R602: 1k, Resistor_THT:R_Axial_DIN0207_L6.3mm_D2.5mm_P10.16mm_Horizontal, F.Cu at (62.9, 140.3)
- added R603: 270, Resistor_THT:R_Axial_DIN0207_L6.3mm_D2.5mm_P10.16mm_Horizontal, F.Cu at (49.1, 144.8)
- added R604: 4k7, Resistor_THT:R_Axial_DIN0207_L6.3mm_D2.5mm_P10.16mm_Horizontal, F.Cu at (62.9, 144.8)
- added R605: 330, Resistor_THT:R_Axial_DIN0207_L6.3mm_D2.5mm_P10.16mm_Horizontal, F.Cu at (49.1, 149.4)
- added R606: 4k7, Resistor_THT:R_Axial_DIN0207_L6.3mm_D2.5mm_P10.16mm_Horizontal, F.Cu at (62.9, 149.4)
- added R607: 180, Resistor_THT:R_Axial_DIN0207_L6.3mm_D2.5mm_P10.16mm_Horizontal, F.Cu at (49.1, 154.0)
- added R608: 4k7, Resistor_THT:R_Axial_DIN0207_L6.3mm_D2.5mm_P10.16mm_Horizontal, F.Cu at (62.9, 154.0)
- added R609: 10k, Resistor_THT:R_Axial_DIN0207_L6.3mm_D2.5mm_P10.16mm_Horizontal, F.Cu at (49.1, 158.6)
- added R610: 220, Resistor_THT:R_Axial_DIN0207_L6.3mm_D2.5mm_P10.16mm_Horizontal, F.Cu at (62.9, 158.6)
- added SW601: TL1105NF250Q, Motor-Controller:SW_E-Switch_TL1105_RightAngle, F.Cu at (41.6, 136.0)
- added U1: Pololu G2 18v25, Motor-Controller:Pololu_G2_18v25_Socket, F.Cu at (155.6, 43.6)
- added U101: R-78B5.0-2.0, Converter_DCDC:Converter_DCDC_RECOM_R-78B-2.0_THT, F.Cu at (116.4, 62.7)
- added U2: ACS758LCB-050B-PFF-T, Sensor_Current:Allegro_CB_PFF, F.Cu at (139.4, 93.5)
- added U201: R-78B5.0-2.0, Converter_DCDC:Converter_DCDC_RECOM_R-78B-2.0_THT, F.Cu at (101.6, 83.4)
- added U301: MCP3208, Package_DIP:DIP-16_W7.62mm_Socket, F.Cu at (49.6, 92.6)
- added U302: LM4040AIZ-2.5, Package_TO_SOT_THT:TO-92_Inline, F.Cu at (90.5, 125.7)
- added U401: MAX3488EEPA, Package_DIP:DIP-8_W7.62mm, F.Cu at (97.2, 124.5)
- added U501: MAX3488EEPA, Package_DIP:DIP-8_W7.62mm, F.Cu at (129.5, 124.5)
- added U601: ESP32-DevKitC-32E, Motor-Controller:ESP32-DevKitC_Socket, F.Cu at (57.3, 41.4)
Other:
- board outline added: 150 x 130 mm
- board text added: "Anordnung 09.10.2026: alle Teile angeordnet, noch ohne Leiterbahnen."
- board text added: "SuAn Motor-Controller V2.0 v00.01"

Commit message: Motor-Controller: J6 feste Degson DG301 statt steckbarer MSTBA; J7 neue Belegung (1 MCY, 2 MCZ, 3 MCB, 4 MCA, 5 RAA, 6 RAB, 7 GND, 8 +5V), J8 entfaellt - Bauteilauswahl 00.24, Stueckliste 00.20, Pruefskript 00.02
Co-Authored-By: Claude Opus 5.5 <noreply@anthropic.com>
Parts:
- removed J8: Steuerhaus 5V, Connector_Phoenix_MSTB:PhoenixContact_MSTBA_2,5_2-G-5,08_1x02_P5.08mm_Horizontal
- J6: footprint Connector_Phoenix_MSTB:PhoenixContact_MSTBA_2,5_2-G-5,08_1x02_P5.08mm_Horizontal -> Motor-Controller:Degson_DG301-5.0-02P
- moved J6 2.50 mm to (90.1, 65.4)
Connections:
- J7 pad 1: /RS422 TinyPilot/A -> /MCY
- J7 pad 2: /RS422 TinyPilot/B -> /MCZ
- J7 pad 3: /RS422 TinyPilot/Z -> /MCB
- J7 pad 4: /RS422 TinyPilot/Y -> /MCA
- J7 pad 5: /RS422 Ruderlage/A -> /RAA
- J7 pad 6: /RS422 Ruderlage/B -> /RAB
- J7 pad 7: /RS422 Ruderlage/Z -> GND
- J7 pad 8: /RS422 Ruderlage/Y -> /+5V_PYPILOT
- R401 pad 1: /RS422 TinyPilot/A -> /MCA
- R401 pad 2: /RS422 TinyPilot/B -> /MCB
- U401 pad 5: /RS422 TinyPilot/Y -> /MCY
- U401 pad 6: /RS422 TinyPilot/Z -> /MCZ
- U401 pad 7: /RS422 TinyPilot/B -> /MCB
- U401 pad 8: /RS422 TinyPilot/A -> /MCA
- U501 pad 5: /RS422 Ruderlage/Y -> /RAA
- U501 pad 6: /RS422 Ruderlage/Z -> /RAB

Commit message: Motor-Controller: Steuerhaus -> Steuerstand; J7 "Steuerstand RS422 fuer TinyPilot"; Bauteile auf der Platine neu angeordnet (Betreiber); KiCad-Neuformatierung
Co-Authored-By: Claude Opus 5.5 <noreply@anthropic.com>
Parts:
- J7: value Steuerhaus RS422 -> Steuerstand RS422
- moved J5 55.4 mm to (179.2, 107.5)
- moved U301 24.3 mm to (54.3, 116.5), turned to 90 degrees
- moved J7 23.9 mm to (179.2, 87.8)
- moved D603 18.2 mm to (44.4, 109.5)
- moved D3 18.2 mm to (44.4, 117.1)
- moved D4 18.2 mm to (44.4, 124.7)
- moved D601 18.2 mm to (44.4, 94.2)
- moved D602 18.2 mm to (44.4, 101.8)
- moved R1 15.8 mm to (50.0, 101.0)
- moved J1 6.37 mm to (50.3, 68.0)
- moved U601 6.30 mm to (55.5, 47.4)
- moved R201 6.25 mm to (101.2, 152.2)
- moved C305 6.25 mm to (156.9, 123.6)
- moved C601 6.25 mm to (115.7, 108.0)
- moved D304 6.25 mm to (94.2, 122.1)
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
Commit message: 12 V zum Steuerstand statt 5 V: eigener Regler 12->5 V (3 A) am Steuerstand
Vom Motorraum gehen 12 V (rot/schwarz) zum Regler am Steuerstand, von dort 5 V
(zweites rot/schwarzes Paar) zur PyPilot-Einheit.
- Systembeschreibung, TODO (Frage 1 geloescht, Frage 18 gekuerzt)
- Motor-Controller: F13 (motorcontroller 00.13), Bauteilauswahl 00.26,
  Blockschaltbild 00.07, Stueckliste 00.21: J7.8 = +12 V hinter D2, ohne
  eigene Sicherung (Betreiber 13.10.2026); zweiter 5-V-Zweig entfernt
- KiCad v00.01: Blatt "5V PyPilot" und 8 Bauteile entfernt; ERC 0 Fehler,
  Paritaet 0, pruefung_blockschaltbild 00.03: 78/78
- Phase 1 Verdrahtungsplaene: Basic (Regler vor TinyPilot), Dual Display
  (Masse zum Regler); Vermerk Einbauort

Co-Authored-By: Claude Opus 5.5 <noreply@anthropic.com>
Parts:
- removed C201, C202, C203: 4u7 50V, Motor-Controller:C_KEMET_C320_L5.1mm_W4.1mm_P2.54mm
- removed D201: rot, Motor-Controller:LED_Dialight_551_RightAngle
- removed F201: 2A T, Fuse:Fuseholder_Cylinder-5x20mm_Schurter_0031_8201_Horizontal_Open
- removed L201: 10uH 2,7A, Inductor_THT:L_Radial_D10.0mm_P5.00mm_Fastron_07P
- removed R201: 4k7, Resistor_THT:R_Axial_DIN0207_L6.3mm_D2.5mm_P10.16mm_Horizontal
- removed U201: R-78B5.0-2.0, Converter_DCDC:Converter_DCDC_RECOM_R-78B-2.0_THT
- J2: footprint Connector_Phoenix_MSTB:PhoenixContact_MSTBA_2,5_2-G-5,08_1x02_P5.08mm_Horizontal -> Motor-Controller:Degson_DG301-5.0-02P
- J7: value Steuerstand RS422 -> Steuerstand RS422 für TinyPilot
- moved J7 67.0 mm to (179.2, 154.8)
- moved J6 40.8 mm to (130.7, 68.8), turned to 90 degrees
- moved U101 27.4 mm to (89.0, 64.3)
- moved U2 20.3 mm to (124.7, 79.6), turned to -90 degrees
- moved J3 16.5 mm to (172.2, 89.3), turned to 180 degrees
- moved J4 9.31 mm to (160.2, 89.3), turned to 180 degrees
- moved R1 5.92 mm to (55.8, 102.0)
- moved R12 5.06 mm to (60.9, 132.2)
- moved R4 5.06 mm to (53.8, 121.4)
- moved Q604 5.06 mm to (75.4, 162.7)
- moved R6 5.06 mm to (53.8, 126.0)
- moved R601 5.06 mm to (53.8, 138.5)
- moved R603 5.06 mm to (53.8, 143.1)
- moved R605 5.06 mm to (53.8, 147.7)
- moved R607 5.06 mm to (53.8, 152.3)
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Connections:
- J7 pad 8: /+5V_PYPILOT -> +12V
