File: 2-motor-controller/hardware/kicad/v00.01/Motor-Controller.kicad_sch (KiCad schematic)
At the start: 5 parts, among them J1 RF300, J2 12V Bordnetz, J5 Pumpe

Commit message: Motor-Controller: Blaetter Messwerterfassung, RS422-Strecke (2x), Rechner und Bedienung; Hauptblatt verbunden, Klemmen zum Steuerhaus; Display-Schaltzeichen
Co-Authored-By: Claude Opus 5.5 <noreply@anthropic.com>
Parts:
- added J7: Steuerhaus RS422, symbol Connector:Screw_Terminal_01x08
- added J8: Steuerhaus 5V, symbol Connector:Screw_Terminal_01x02
Connections:
- net +5V_PYPILOT: now also J8.1 (Pin_1)
- net GND: now also J8.2 (Pin_2)
- net Endstufe/KLEMME_A renamed KLEMME_A
- net Endstufe/KLEMME_B renamed KLEMME_B
- new net RS422 Ruderlage/A: J7.5 (Pin_5)
- new net RS422 Ruderlage/B: J7.6 (Pin_6)
- new net RS422 Ruderlage/Y: J7.8 (Pin_8)
- new net RS422 Ruderlage/Z: J7.7 (Pin_7)
- new net RS422 TinyPilot/A: J7.1 (Pin_1)
- new net RS422 TinyPilot/B: J7.2 (Pin_2)
- new net RS422 TinyPilot/Y: J7.4 (Pin_4)
- new net RS422 TinyPilot/Z: J7.3 (Pin_3)
- no-connect marks 0 -> 1
Other:
- added sheet Messwerterfassung (Messwerterfassung.kicad_sch)
- added sheet RS422 Ruderlage (RS422-Strecke.kicad_sch)
- added sheet RS422 TinyPilot (RS422-Strecke.kicad_sch)
- added sheet Rechner und Bedienung (Rechner.kicad_sch)
- note added: "J7 MSTBA 2,5/8 zum Steuerhaus, Belegung wie J9 der RF300-Interfaceplatine: 1–4 TinyPilot A+, B−, Z−, Y+; 5–8 Ruderlage A+, B−, Z−, Y+ (A/B empfangen, Y/Z senden). J8 MSTBA 2,5/2: 5 V für die PyPilot-Einheit (rot/schwarz)."
- note added: "Messwerte: Spannung an den Pumpenklemmen, Bordspannung, Strom (Pololu und Hall-Sensor), Temperatur der Endstufe. Rechner: Pumpe ansteuern, überwachen, Display, Leuchtdioden, Taster."

Commit message: Motor-Controller: alle Blaetter nach den Zeichenregeln (Rahmen, Gruppen), 5-V-Zweig mit 2 x 4,7 uF, Titelfelder Version 00.01; Pruefung gegen Blockschaltbild 78/78
Co-Authored-By: Claude Opus 5.5 <noreply@anthropic.com>
Other:
- company: (none) -> SuAn-Autopilot-Projekt
- title: (none) -> Motor-Controller V2.0 – Hauptblatt
Changed lines of the file:
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@@
 	(generator_version "10.0")
 	(paper "A3")
+	(title_block
+		(title "Motor-Controller V2.0 – Hauptblatt")
+		(date "2026-10-09")
+		(rev "00.01")
+		(company "SuAn-Autopilot-Projekt")
+	)
 	(rectangle
 		(start 13.97 11.43)

Commit message: Motor-Controller: Loetbilder zugeordnet (eigene: Dialight 551, TL1105, KEMET C320, Display-Leiste), Platine 150 x 130 mm mit allen 94 Teilen angeordnet - Bauteilauswahl 00.23, Anforderungen 00.11, Stueckliste 00.19
Co-Authored-By: Claude Opus 5.5 <noreply@anthropic.com>
Parts:
- J7: footprint (none) -> Connector_Phoenix_MSTB:PhoenixContact_MSTBA_2,5_8-G-5,08_1x08_P5.08mm_Horizontal
- J8: footprint (none) -> Connector_Phoenix_MSTB:PhoenixContact_MSTBA_2,5_2-G-5,08_1x02_P5.08mm_Horizontal
Changed lines of the file:
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@@
 			)
 		)
-		(property "Footprint" ""
+		(property "Footprint" "Connector_Phoenix_MSTB:PhoenixContact_MSTBA_2,5_2-G-5,08_1x02_P5.08mm_Horizontal"
 			(at 397.51 93.98 0)
 			(hide yes)
@@
 			)
 		)
-		(property "Footprint" ""
+		(property "Footprint" "Connector_Phoenix_MSTB:PhoenixContact_MSTBA_2,5_8-G-5,08_1x08_P5.08mm_Horizontal"
 			(at 397.51 147.32 0)
 			(hide yes)

Commit message: Motor-Controller: J6 feste Degson DG301 statt steckbarer MSTBA; J7 neue Belegung (1 MCY, 2 MCZ, 3 MCB, 4 MCA, 5 RAA, 6 RAB, 7 GND, 8 +5V), J8 entfaellt - Bauteilauswahl 00.24, Stueckliste 00.20, Pruefskript 00.02
Co-Authored-By: Claude Opus 5.5 <noreply@anthropic.com>
Parts:
- removed J8: Steuerhaus 5V, Connector_Phoenix_MSTB:PhoenixContact_MSTBA_2,5_2-G-5,08_1x02_P5.08mm_Horizontal, symbol Connector:Screw_Terminal_01x02
Connections:
- net RS422 Ruderlage/Y is gone; now on net +5V_PYPILOT: J7.8 (Pin_8)
- net RS422 Ruderlage/Z is gone; now on net GND: J7.7 (Pin_7)
- net RS422 Ruderlage/A: no longer J7.5 (Pin_5)
- net RS422 Ruderlage/B: no longer J7.6 (Pin_6)
- net RS422 TinyPilot/A renamed MCY
- net RS422 TinyPilot/B renamed MCZ
- net RS422 TinyPilot/Y renamed MCA
- net RS422 TinyPilot/Z renamed MCB
- new net RAA: J7.5 (Pin_5)
- new net RAB: J7.6 (Pin_6)
- no-connect marks 1 -> 3
Other:
- note added: "J7 MSTBA 2,5/8 zum Steuerhaus (Betreiber, 09.10.2026): 1 MCY, 2 MCZ (Controller sendet zum TinyPilot); 3 MCB, 4 MCA (TinyPilot sendet zum Controller); 5 RAA, 6 RAB (NMEA-Ruderlage zum TinyPilot, nur Senden); 7 GND, 8 +5 V für die PyPilot-Einheit."
- note removed: "J7 MSTBA 2,5/8 zum Steuerhaus, Belegung wie J9 der RF300-Interfaceplatine: 1–4 TinyPilot A+, B−, Z−, Y+; 5–8 Ruderlage A+, B−, Z−, Y+ (A/B empfangen, Y/Z senden). J8 MSTBA 2,5/2: 5 V für die PyPilot-Einheit (rot/schwarz)."

Commit message: Motor-Controller: Steuerhaus -> Steuerstand; J7 "Steuerstand RS422 fuer TinyPilot"; Bauteile auf der Platine neu angeordnet (Betreiber); KiCad-Neuformatierung
Co-Authored-By: Claude Opus 5.5 <noreply@anthropic.com>
Parts:
- J7: value Steuerhaus RS422 -> Steuerstand RS422 für TinyPilot

Commit message: 12 V zum Steuerstand statt 5 V: eigener Regler 12->5 V (3 A) am Steuerstand
Vom Motorraum gehen 12 V (rot/schwarz) zum Regler am Steuerstand, von dort 5 V
(zweites rot/schwarzes Paar) zur PyPilot-Einheit.
- Systembeschreibung, TODO (Frage 1 geloescht, Frage 18 gekuerzt)
- Motor-Controller: F13 (motorcontroller 00.13), Bauteilauswahl 00.26,
  Blockschaltbild 00.07, Stueckliste 00.21: J7.8 = +12 V hinter D2, ohne
  eigene Sicherung (Betreiber 13.10.2026); zweiter 5-V-Zweig entfernt
- KiCad v00.01: Blatt "5V PyPilot" und 8 Bauteile entfernt; ERC 0 Fehler,
  Paritaet 0, pruefung_blockschaltbild 00.03: 78/78
- Phase 1 Verdrahtungsplaene: Basic (Regler vor TinyPilot), Dual Display
  (Masse zum Regler); Vermerk Einbauort

Co-Authored-By: Claude Opus 5.5 <noreply@anthropic.com>
Parts:
- J2: footprint Connector_Phoenix_MSTB:PhoenixContact_MSTBA_2,5_2-G-5,08_1x02_P5.08mm_Horizontal -> Motor-Controller:Degson_DG301-5.0-02P
Connections:
- net +5V_PYPILOT is gone; now on net +12V: J7.8 (Pin_8)
Other:
- removed sheet 5V PyPilot
- note added: "J7 MSTBA 2,5/8 zum Steuerhaus (Betreiber, 09.10.2026): 1 MCY, 2 MCZ (Controller sendet zum TinyPilot); 3 MCB, 4 MCA (TinyPilot sendet zum Controller); 5 RAA, 6 RAB (NMEA-Ruderlage zum TinyPilot, nur Senden); 7 GND, 8 +12 V für die PyPilot-Einheit (hinter D2, ohne eigene Sicherung, Betreiber 13.10.2026); die 5 V macht ein eigener Regler am Steuerstand."
- note removed: "J7 MSTBA 2,5/8 zum Steuerhaus (Betreiber, 09.10.2026): 1 MCY, 2 MCZ (Controller sendet zum TinyPilot); 3 MCB, 4 MCA (TinyPilot sendet zum Controller); 5 RAA, 6 RAB (NMEA-Ruderlage zum TinyPilot, nur Senden); 7 GND, 8 +5 V für die PyPilot-Einheit."
Changed lines of the file:
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@@
 		)
 	)
-	(text "J7 MSTBA 2,5/8 zum Steuerhaus (Betreiber, 09.10.2026):\n1 MCY, 2 MCZ (Controller sendet zum TinyPilot); 3 MCB, 4 MCA (TinyPilot sendet zum Controller);\n5 RAA, 6 RAB (NMEA-Ruderlage zum TinyPilot, nur Senden); 7 GND, 8 +5 V für die PyPilot-Einheit."
+	(text "J7 MSTBA 2,5/8 zum Steuerhaus (Betreiber, 09.10.2026):\n1 MCY, 2 MCZ (Controller sendet zum TinyPilot); 3 MCB, 4 MCA (TinyPilot sendet zum Controller);\n5 RAA, 6 RAB (NMEA-Ruderlage zum TinyPilot, nur Senden); 7 GND, 8 +12 V für die PyPilot-Einheit (hinter D2, ohne eigene Sicherung, Betreiber 13.10.2026);\ndie 5 V macht ein eigener Regler am Steuerstand."
 		(exclude_from_sim no)
 		(at 265.43 198.12 0)
@@
 	(wire
 		(pts
-			(xy 322.58 93.98) (xy 345.44 93.98)
-		)
-		(stroke
-			(width 0)
-			(type default)
-		)
-	)
-	(wire
-		(pts
 			(xy 149.86 57.15) (xy 144.78 57.15)
 		)
@@
 	(wire
 		(pts
-			(xy 292.1 93.98) (xy 287.02 93.98)
-		)
-		(stroke
-			(width 0)
-			(type default)
-		)
-	)
-	(wire
-		(pts
 			(xy 330.2 147.32) (xy 335.28 147.32)
 		)
@@
 	(wire
 		(pts
-			(xy 287.02 93.98) (xy 287.02 91.44)
-		)
-		(stroke
-			(width 0)
-			(type default)
-		)
-	)
-	(wire
-		(pts
 			(xy 144.78 57.15) (xy 144.78 54.61)
 		)
@@
 	(wire
 		(pts
-			(xy 287.02 104.14) (xy 287.02 106.68)
-		)
-		(stroke
-			(width 0)
-			(type default)
-		)
-	)
-	(wire
-		(pts
 			(xy 39.37 88.9) (xy 39.37 91.44)
 		)
@@
 		)
 	)
-	(wire
-		(pts
-			(xy 292.1 104.14) (xy 287.02 104.14)
-		)
-		(stroke
-			(width 0)
-			(type default)
-		)
-	)
 	(label "HALL"
 		(at 335.28 35.56 0)
@@
 		)
 	)
-	(label "+5V_PYPILOT"
-		(at 345.44 93.98 0)
-		(effects
-			(font
-				(size 1.27 1.27)
-			)
-			(justify left bottom)
-		)
-	)
-	(label "+5V_PYPILOT"
-		(at 387.35 157.48 180)
-		(effects
-			(font
-				(size 1.27 1.27)
-			)
-			(justify right bottom)
-		)
-	)
 	(label "MCB"
 		(at 387.35 144.78 180)
@@
 	(symbol
 		(lib_id "power:+12V")
-		(at 287.02 91.44 0)
+		(at 387.35 157.48 90)
 		(unit 1)
 		(body_style 1)
@@
 		(dnp no)
 		(property "Reference" "#PWR06"
-			(at 287.02 88.9 0)
+			(at 387.35 157.48 0)
 			(hide yes)
 			(show_name no)
@@
 		)
 		(property "Value" "+12V"
-			(at 287.02 87.63 0)
+			(at 383.54 157.48 90)
 			(show_name no)
 			(do_not_autoplace no)
@@
 					(size 1.27 1.27)
 				)
+				(justify left)
 			)
 		)
 		(property "Footprint" ""
-			(at 287.02 91.44 0)
+			(at 387.35 157.48 0)
 			(hide yes)
 			(show_name no)
@@
 		)
 		(property "Datasheet" ""
-			(at 287.02 91.44 0)
+			(at 387.35 157.48 0)
 			(hide yes)
 			(show_name no)
@@
 		)
 		(property "Description" "Power symbol creates a global label with name \"+12V\""
-			(at 287.02 91.44 0)
+			(at 387.35 157.48 0)
 			(hide yes)
 			(show_name no)
@@
 	(symbol
 		(lib_id "power:GND")
-		(at 287.02 106.68 0)
-		(unit 1)
-		(body_style 1)
-		(exclude_from_sim no)
-		(in_bom yes)
-		(on_board yes)
-		(in_pos_files yes)
-		(dnp no)
-		(property "Reference" "#PWR07"
-			(at 287.02 104.14 0)
-			(hide yes)
-			(show_name no)
-			(do_not_autoplace no)
-			(effects
-				(font
-					(size 1.27 1.27)
-				)
-			)
-		)
-		(property "Value" "GND"
-			(at 287.02 109.22 0)
-			(show_name no)
-			(do_not_autoplace no)
-			(effects
-				(font
-					(size 1.27 1.27)
-				)
-			)
-		)
-		(property "Footprint" ""
-			(at 287.02 106.68 0)
-			(hide yes)
-			(show_name no)
-			(do_not_autoplace no)
-			(effects
-				(font
-					(size 1.27 1.27)
-				)
-			)
-		)
-		(property "Datasheet" ""
-			(at 287.02 106.68 0)
-			(hide yes)
-			(show_name no)
-			(do_not_autoplace no)
-			(effects
-				(font
-					(size 1.27 1.27)
-				)
-			)
-		)
-		(property "Description" "Power symbol creates a global label with name \"GND\" , ground"
-			(at 287.02 106.68 0)
-			(hide yes)
-			(show_name no)
-			(do_not_autoplace no)
-			(effects
-				(font
-					(size 1.27 1.27)
-				)
-			)
-		)
-		(pin "1"
-		)
-		(instances
-			(project "Motor-Controller"
-				(path "/255b263c-8a60-4b67-92ab-70f539cf8eaf"
-					(reference "#PWR07")
-					(unit 1)
-				)
-			)
-		)
-	)
-	(symbol
-		(lib_id "power:GND")
 		(at 39.37 91.44 0)
 		(unit 1)
@@
 			)
 		)
-		(property "Footprint" "Connector_Phoenix_MSTB:PhoenixContact_MSTBA_2,5_2-G-5,08_1x02_P5.08mm_Horizontal"
+		(property "Footprint" "Motor-Controller:Degson_DG301-5.0-02P"
 			(at 21.59 21.59 0)
 			(hide yes)
@@
 			(project "Motor-Controller"
 				(path "/255b263c-8a60-4b67-92ab-70f539cf8eaf"
-					(page "9")
+					(page "8")
 				)
 			)
@@
 			(project "Motor-Controller"
 				(path "/255b263c-8a60-4b67-92ab-70f539cf8eaf"
-					(page "6")
+					(page "5")
 				)
 			)
@@
 			(project "Motor-Controller"
 				(path "/255b263c-8a60-4b67-92ab-70f539cf8eaf"
-					(page "7")
-				)
-			)
-		)
-	)
-	(sheet
-		(at 292.1 88.9)
-		(size 30.48 20.32)
-		(exclude_from_sim no)
-		(in_bom yes)
-		(on_board yes)
-		(dnp no)
-		(fields_autoplaced yes)
-		(stroke
-			(width 0.0006)
-			(type solid)
-		)
-		(fill
-			(color 0 0 0 0)
-		)
-		(property "Sheetname" "5V PyPilot"
-			(at 294.64 87.63 0)
-			(show_name no)
-			(do_not_autoplace no)
-			(effects
-				(font
-					(size 1.27 1.27)
-				)
-				(justify left bottom)
-			)
-		)
-		(property "Sheetfile" "5V-Zweig.kicad_sch"
-			(at 294.64 110.49 0)
-			(show_name no)
-			(do_not_autoplace no)
-			(effects
-				(font
-					(size 1.27 1.27)
-				)
-				(justify left top)
-			)
-		)
-		(pin "+12V" input
-			(at 292.1 93.98 180)
-			(effects
-				(font
-					(size 1.27 1.27)
-				)
-				(justify left)
-			)
-		)
-		(pin "GND" input
-			(at 292.1 104.14 180)
-			(effects
-				(font
-					(size 1.27 1.27)
-				)
-				(justify left)
-			)
-		)
-		(pin "+5V" output
-			(at 322.58 93.98 0)
-			(effects
-				(font
-					(size 1.27 1.27)
-				)
-				(justify right)
-			)
-		)
-		(instances
-			(project "Motor-Controller"
-				(path "/255b263c-8a60-4b67-92ab-70f539cf8eaf"
-					(page "4")
+					(page "6")
 				)
 			)
@@
 			(project "Motor-Controller"
 				(path "/255b263c-8a60-4b67-92ab-70f539cf8eaf"
-					(page "5")
+					(page "4")
 				)
 			)
@@
 			(project "Motor-Controller"
 				(path "/255b263c-8a60-4b67-92ab-70f539cf8eaf"
-					(page "8")
+					(page "7")
 				)
 			)
