File: 10-Robertson-Bedieneinheit/robnet-analyse/hardware/kicad/v00.01/Rechner.kicad_sch (KiCad schematic)
At the start: 1 part, among them J5 Raspberry Pi Zero 2 W

Commit message: Robnet-Analyse Platine v00.01: Bauteile platziert, JLCPCB-Regeln, Leiterbahnklassen, 3D-Modelle zugeordnet
- Bauformen gegen Datenblatt geprueft: BAT85 DO-35, 1.5KE20A DO-201, J5 = Zero kopfueber mit Umriss und Aufdruck
- platine_erzeugen/robnet_platine.py: Lage, Aufdruck, Regeln, Klassen (Vsys+ 1,5 mm / Versorgung 1,0 mm), 3D-Modelle;
  DRC nur Aufdruck an der Kante und offene Verbindungen, Abgleich Schaltplan 0
- 3d-modelle/eigene_modelle.py und kicad_lage.py (STEP-Dateien selbst nicht in Git)
- Bauteilauswahl 00.13, Konzept 00.29, bom.csv 00.06

Co-Authored-By: Claude Opus 5.5 <noreply@anthropic.com>
Parts:
- J5: footprint Connector_PinSocket_2.54mm:PinSocket_2x20_P2.54mm_Vertical -> Robnet-Analyse:Raspberry_Pi_Zero_kopfueber
Changed lines of the file:
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@@
 			)
 		)
-		(property "Footprint" "Connector_PinSocket_2.54mm:PinSocket_2x20_P2.54mm_Vertical"
+		(property "Footprint" "Robnet-Analyse:Raspberry_Pi_Zero_kopfueber"
 			(at 148.59 101.6 0)
 			(hide yes)
