File: 10-Robertson-Bedieneinheit/robnet-analyse/hardware/kicad/v00.01/Versorgung.kicad_sch (KiCad schematic)
At the start: 10 parts, among them U3 R-78B5.0-2.0

Commit message: Robnet-Analyse Platine v00.01: Bauteile platziert, JLCPCB-Regeln, Leiterbahnklassen, 3D-Modelle zugeordnet
- Bauformen gegen Datenblatt geprueft: BAT85 DO-35, 1.5KE20A DO-201, J5 = Zero kopfueber mit Umriss und Aufdruck
- platine_erzeugen/robnet_platine.py: Lage, Aufdruck, Regeln, Klassen (Vsys+ 1,5 mm / Versorgung 1,0 mm), 3D-Modelle;
  DRC nur Aufdruck an der Kante und offene Verbindungen, Abgleich Schaltplan 0
- 3d-modelle/eigene_modelle.py und kicad_lage.py (STEP-Dateien selbst nicht in Git)
- Bauteilauswahl 00.13, Konzept 00.29, bom.csv 00.06

Co-Authored-By: Claude Opus 5.5 <noreply@anthropic.com>
Parts:
- D2: footprint Diode_THT:D_DO-201AE_P15.24mm_Horizontal -> Diode_THT:D_DO-201_P15.24mm_Horizontal
Changed lines of the file:
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@@
 			)
 		)
-		(property "Footprint" "Diode_THT:D_DO-201AE_P15.24mm_Horizontal"
+		(property "Footprint" "Diode_THT:D_DO-201_P15.24mm_Horizontal"
 			(at 73.66 87.63 90)
 			(hide yes)
