File: 10-Robertson-Bedieneinheit/robnet-analyse/hardware/smd/kicad/v00.01/platine_erzeugen/Robnet-Analyse_platziert.kicad_pcb (KiCad board)
At the start: 2 copper layers, 100 x 100 mm, 71 parts, among them J1 MSTBA 6-pol., J2 MSTBA 2-pol., J3 MSTBA 6-pol., J4 Messpunkte, J5 Raspberry Pi Zero 2 W, U1 MAX3488EEPA, U2 MCP3208-CI/P, U3 R-78B5.0-2.0, U4 LM4040AIZ-2.5, U6 MCP3208-CI/P

Commit message: Robnet-Analyse Linie B: Leiterbahnen Gruppe 2 (Adern J1 -> Jumper -> J3)
- Platzierung 00.04: R31-R39 um 180 Grad (Ader aussen), Kanalzeilen in Kanalfolge
  der Wandler (CH0 unten)
- Bahnen 00.02: Seite J300 ueber J1 und durch die Gasse zu den Teilern, Seite
  Bedieneinheit rechts herum und in Boegen unter J3 durch (keine Kreuzung trotz
  gespiegelter Klemmen); JP2, J4, R23, R21; 11 Durchkontaktierungen
- 3,3 V unten zwischen die Kanalbloecke verlegt; Schalter --neue-lage
- DRC ohne Fehler, Abgleich 0; Konzept 00.40, Bauteilauswahl SMD 00.12

Co-Authored-By: Claude Opus 5.5 <noreply@anthropic.com>
Parts:
- moved D11 24.0 mm to (54.9, 56.5)
- moved D16 24.0 mm to (54.9, 32.5)
- moved R11 24.0 mm to (50.5, 56.5)
- moved R12 24.0 mm to (59.9, 56.5)
- moved R21 24.0 mm to (50.5, 32.5)
- moved R22 24.0 mm to (59.9, 32.5)
- moved D31 19.2 mm to (54.9, 80.7)
- moved D35 19.2 mm to (54.9, 61.5)
- moved R31 19.2 mm to (50.5, 80.7), turned to 180 degrees
- moved R32 19.2 mm to (59.9, 80.7)
- moved R39 19.2 mm to (50.5, 61.5), turned to 180 degrees
- moved R40 19.2 mm to (59.9, 61.5)
- moved D12 14.4 mm to (54.9, 51.7)
- moved D15 14.4 mm to (54.9, 37.3)
- moved R13 14.4 mm to (50.5, 51.7)
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