File: 10-Robertson-Bedieneinheit/robnet-analyse/hardware/smd/kicad/v00.01/platine_erzeugen/Robnet-Analyse_platziert.kicad_pcb (KiCad board)
At the start: 2 copper layers, 100 x 100 mm, 71 parts, among them J1 MSTBA 6-pol., J2 MSTBA 2-pol., J3 MSTBA 6-pol., J4 Messpunkte, J5 Raspberry Pi Zero 2 W, U1 MAX3488EEPA, U2 MCP3208-CI/P, U3 R-78B5.0-2.0, U4 LM4040AIZ-2.5, U6 MCP3208-CI/P

Commit message: Robnet-Analyse Linie B: Messbereich 20 V, Fertigungsdateien (Schritt 4), Beschaffungslisten
- Teiler 18 -> 13 kOhm (C17455, Preferred): Messbereich ~21,7 V; Vsys bleibt ~33 V
- Selbst geloetete Teile (18) in Schaltplan und Platine aus Stueck- und
  Positionsliste genommen; ERC 0, Pruefskript 87/87, DRC ohne Meldung
- production/: Gerber, bom.csv, positions.csv (Fabrication Toolkit 5.3.1),
  geprueft mit pruefung_fertigung.py (49 Teile, 0 Fehler)
- bom_tht_beschaffung.csv (2 Platinen) und bom_zubehoer.csv, je zwei Haendler
- Ablauf SMD 00.03 (Toolkit-Installation, Aufruf ohne Oberflaeche), TODO 23
  (Linie A ebenfalls 13 kOhm), Konzept 00.46, Blockschaltbild 00.17

Co-Authored-By: Claude Opus 5.5 <noreply@anthropic.com>
Parts:
- R12, R14, R18, R20, R22, R34, R36, R38, R40: value 18k 1% -> 13k 1%
