File: 10-Robertson-Bedieneinheit/robnet-analyse/hardware/smd/kicad/v00.01/Bus-Empfaenger.kicad_sch (KiCad schematic)
At the start: 6 parts, among them U1 MAX3488EEPA

Commit message: Robnet-Analyse Linie B: Messbereich 20 V, Fertigungsdateien (Schritt 4), Beschaffungslisten
- Teiler 18 -> 13 kOhm (C17455, Preferred): Messbereich ~21,7 V; Vsys bleibt ~33 V
- Selbst geloetete Teile (18) in Schaltplan und Platine aus Stueck- und
  Positionsliste genommen; ERC 0, Pruefskript 87/87, DRC ohne Meldung
- production/: Gerber, bom.csv, positions.csv (Fabrication Toolkit 5.3.1),
  geprueft mit pruefung_fertigung.py (49 Teile, 0 Fehler)
- bom_tht_beschaffung.csv (2 Platinen) und bom_zubehoer.csv, je zwei Haendler
- Ablauf SMD 00.03 (Toolkit-Installation, Aufruf ohne Oberflaeche), TODO 23
  (Linie A ebenfalls 13 kOhm), Konzept 00.46, Blockschaltbild 00.17

Co-Authored-By: Claude Opus 5.5 <noreply@anthropic.com>
Parts:
- JP1, JP2, U1: now left out of the parts list
