File: 10-Robertson-Bedieneinheit/robnet-analyse/hardware/smd/kicad/v00.01/Messung.kicad_sch (KiCad schematic)
At the start: 42 parts, among them U2 MCP3208-CI/P, U4 LM4040AIZ-2.5, U6 MCP3208-CI/P

Commit message: Robnet-Analyse Linie B: Messbereich 20 V, Fertigungsdateien (Schritt 4), Beschaffungslisten
- Teiler 18 -> 13 kOhm (C17455, Preferred): Messbereich ~21,7 V; Vsys bleibt ~33 V
- Selbst geloetete Teile (18) in Schaltplan und Platine aus Stueck- und
  Positionsliste genommen; ERC 0, Pruefskript 87/87, DRC ohne Meldung
- production/: Gerber, bom.csv, positions.csv (Fabrication Toolkit 5.3.1),
  geprueft mit pruefung_fertigung.py (49 Teile, 0 Fehler)
- bom_tht_beschaffung.csv (2 Platinen) und bom_zubehoer.csv, je zwei Haendler
- Ablauf SMD 00.03 (Toolkit-Installation, Aufruf ohne Oberflaeche), TODO 23
  (Linie A ebenfalls 13 kOhm), Konzept 00.46, Blockschaltbild 00.17

Co-Authored-By: Claude Opus 5.5 <noreply@anthropic.com>
Parts:
- R12, R14, R18, R20, R22, R34, R36, R38, R40: value 18k 1% -> 13k 1%; LCSC Part # C17506 -> C17455
- U2, U4, U6: now left out of the parts list
Other:
- note added: "Teiler 100 k / 13 k (bis ~21,7 V), Vsys+ 100 k / 8,2 k (bis ~33 V), alle 1 % (UNI-ROYAL 0805). Je Kanal eine BAT54S nach +3,3 V und Masse. Bus-Kanäle ohne Glättung. Last je Ader ~113 kΩ. U2, U6 MCP3208 (12 Bit, THT-Fassung), Referenz U4 LM4040 2,5 V (TO-92) für beide. Alarm an den Zero (GPIO27): ALARM_J über 100 k / 180 k, 4,8 V → ~3,1 V, BAT54S nach +3,3 V und Masse."
- note removed: "Teiler 100 k / 18 k (bis ~16 V), Vsys+ 100 k / 8,2 k (bis ~33 V), alle 1 % (UNI-ROYAL 0805). Je Kanal eine BAT54S nach +3,3 V und Masse. Bus-Kanäle ohne Glättung. Last je Ader ~118 kΩ. U2, U6 MCP3208 (12 Bit, THT-Fassung), Referenz U4 LM4040 2,5 V (TO-92) für beide. Alarm an den Zero (GPIO27): ALARM_J über 100 k / 180 k, 4,8 V → ~3,1 V, BAT54S nach +3,3 V und Masse."
