File: 10-Robertson-Bedieneinheit/robnet-analyse/hardware/smd/kicad/v00.01/Robnet-Analyse.kicad_sch (KiCad schematic)
At the start: 9 parts, among them J1 MSTBA 6-pol., J2 MSTBA 2-pol., J3 MSTBA 6-pol., J4 Messpunkte

Commit message: Robnet-Analyse Linie B: Messbereich 20 V, Fertigungsdateien (Schritt 4), Beschaffungslisten
- Teiler 18 -> 13 kOhm (C17455, Preferred): Messbereich ~21,7 V; Vsys bleibt ~33 V
- Selbst geloetete Teile (18) in Schaltplan und Platine aus Stueck- und
  Positionsliste genommen; ERC 0, Pruefskript 87/87, DRC ohne Meldung
- production/: Gerber, bom.csv, positions.csv (Fabrication Toolkit 5.3.1),
  geprueft mit pruefung_fertigung.py (49 Teile, 0 Fehler)
- bom_tht_beschaffung.csv (2 Platinen) und bom_zubehoer.csv, je zwei Haendler
- Ablauf SMD 00.03 (Toolkit-Installation, Aufruf ohne Oberflaeche), TODO 23
  (Linie A ebenfalls 13 kOhm), Konzept 00.46, Blockschaltbild 00.17

Co-Authored-By: Claude Opus 5.5 <noreply@anthropic.com>
Parts:
- J1, J2, J3, J4, JP3, JP4, JP5, JP6, JP7: now left out of the parts list
Changed lines of the file:
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@@
 		(body_style 1)
 		(exclude_from_sim no)
-		(in_bom yes)
+		(in_bom no)
 		(on_board yes)
-		(in_pos_files yes)
+		(in_pos_files no)
 		(dnp no)
 		(property "Reference" "J1"
@@
 		(body_style 1)
 		(exclude_from_sim no)
-		(in_bom yes)
+		(in_bom no)
 		(on_board yes)
-		(in_pos_files yes)
+		(in_pos_files no)
 		(dnp no)
 		(property "Reference" "J3"
@@
 		(body_style 1)
 		(exclude_from_sim no)
-		(in_bom yes)
+		(in_bom no)
 		(on_board yes)
-		(in_pos_files yes)
+		(in_pos_files no)
 		(dnp no)
 		(property "Reference" "JP4"
@@
 		(body_style 1)
 		(exclude_from_sim no)
-		(in_bom yes)
+		(in_bom no)
 		(on_board yes)
-		(in_pos_files yes)
+		(in_pos_files no)
 		(dnp no)
 		(property "Reference" "JP3"
@@
 		(body_style 1)
 		(exclude_from_sim no)
-		(in_bom yes)
+		(in_bom no)
 		(on_board yes)
-		(in_pos_files yes)
+		(in_pos_files no)
 		(dnp no)
 		(property "Reference" "JP5"
@@
 		(body_style 1)
 		(exclude_from_sim no)
-		(in_bom yes)
+		(in_bom no)
 		(on_board yes)
-		(in_pos_files yes)
+		(in_pos_files no)
 		(dnp no)
 		(property "Reference" "JP6"
@@
 		(body_style 1)
 		(exclude_from_sim no)
-		(in_bom yes)
+		(in_bom no)
 		(on_board yes)
-		(in_pos_files yes)
+		(in_pos_files no)
 		(dnp no)
 		(property "Reference" "JP7"
@@
 		(in_bom no)
 		(on_board no)
-		(in_pos_files yes)
+		(in_pos_files no)
 		(dnp no)
 		(property "Reference" "#PWR001"
@@
 		(body_style 1)
 		(exclude_from_sim no)
-		(in_bom yes)
+		(in_bom no)
 		(on_board yes)
-		(in_pos_files yes)
+		(in_pos_files no)
 		(dnp no)
 		(property "Reference" "J4"
@@
 		(in_bom no)
 		(on_board no)
-		(in_pos_files yes)
+		(in_pos_files no)
 		(dnp no)
 		(property "Reference" "#PWR002"
@@
 		(body_style 1)
 		(exclude_from_sim no)
-		(in_bom yes)
+		(in_bom no)
 		(on_board yes)
-		(in_pos_files yes)
+		(in_pos_files no)
 		(dnp no)
 		(property "Reference" "J2"
@@
 		(in_bom no)
 		(on_board no)
-		(in_pos_files yes)
+		(in_pos_files no)
 		(dnp no)
 		(property "Reference" "#PWR003"
@@
 		(in_bom no)
 		(on_board no)
-		(in_pos_files yes)
+		(in_pos_files no)
 		(dnp no)
 		(property "Reference" "#FLG01"
@@
 		(in_bom no)
 		(on_board no)
-		(in_pos_files yes)
+		(in_pos_files no)
 		(dnp no)
 		(property "Reference" "#PWR004"
@@
 		(in_bom no)
 		(on_board no)
-		(in_pos_files yes)
+		(in_pos_files no)
 		(dnp no)
 		(property "Reference" "#PWR005"
@@
 		(in_bom no)
 		(on_board no)
-		(in_pos_files yes)
+		(in_pos_files no)
 		(dnp no)
 		(property "Reference" "#PWR006"
@@
 		(in_bom no)
 		(on_board no)
-		(in_pos_files yes)
+		(in_pos_files no)
 		(dnp no)
 		(property "Reference" "#PWR007"
